Commit message: se arregla orientacion del sdf model axioma

File: axioma_ws/src/axioma_urdf/urdf/robot_axioma.urdf (robot description, URDF)
Before this commit: robot sam_bot, 6 links, 5 joints
Links:
- removed link world
Joints:
- removed joint fixed
- joint base_to_wheel3: axis 0 1 0 -> 0 -1 0
- joint base_to_wheel4: axis 0 1 0 -> 0 -1 0

Commit message: update sdf and urdf

File: axioma_ws/src/axioma_urdf/urdf/robot_axioma.urdf (robot description, URDF)
Before this commit: robot sam_bot, 5 links, 4 joints
Links:
- link base_link: geometry collision mesh filename=package://axioma_urdf/meshes/collision/chasiss.dae scale=1 1 1; visual mesh filename=package://axioma_urdf/meshes/visual/chasiss.stl scale=1 1 1
- link wheel_1: geometry collision mesh filename=package://axioma_urdf/meshes/collision/wheel.dae scale=1 1 1; visual mesh filename=package://axioma_urdf/meshes/visual/wheel.stl scale=1 1 1
- link wheel_2: geometry collision mesh filename=package://axioma_urdf/meshes/collision/wheel.dae scale=1 1 1; visual mesh filename=package://axioma_urdf/meshes/visual/wheel.stl scale=1 1 1
- link wheel_3: geometry collision mesh filename=package://axioma_urdf/meshes/collision/wheel.dae scale=1 1 1; visual mesh filename=package://axioma_urdf/meshes/visual/wheel.stl scale=1 1 1
- link wheel_4: geometry collision mesh filename=package://axioma_urdf/meshes/collision/wheel.dae scale=1 1 1; visual mesh filename=package://axioma_urdf/meshes/visual/wheel.stl scale=1 1 1
Joints:
- joint base_to_wheel1: origin xyz=0.06442 0.07385 0.04068 rpy=0 0 0 -> xyz=0.06442 0.07385 0.04068 rpy=3.141516 0 0
- joint base_to_wheel2: origin xyz=-0.071224 0.07385 0.04068 rpy=0 0 0 -> xyz=-0.071224 0.07385 0.04068 rpy=3.141516 0 0
- joint base_to_wheel3: origin xyz=-0.071224 -0.0625 0.04068 rpy=0 0 -3.14159 -> xyz=-0.071224 -0.0625 0.04068 rpy=0 0 0
- joint base_to_wheel4: origin xyz=0.064423 -0.0625 0.04068 rpy=0 0 -3.14159 -> xyz=0.064423 -0.0625 0.04068 rpy=0 0 0

Commit message: navegacion 2

File: axioma_ws/src/axioma_urdf/urdf/robot_axioma.urdf (robot description, URDF)
Before this commit: robot sam_bot, 5 links, 4 joints
Links:
- link base_link: geometry collision mesh filename=package://axioma_urdf/meshes/collision/chasis.dae scale=1 1 1; visual mesh filename=package://axioma_urdf/meshes/visual/chasis.stl scale=1 1 1
- link wheel_1: geometry collision mesh filename=package://axioma_urdf/meshes/collision/llanta.dae scale=1 1 1; visual mesh filename=package://axioma_urdf/meshes/visual/llanta.stl scale=1 1 1
- link wheel_2: geometry collision mesh filename=package://axioma_urdf/meshes/collision/llanta.dae scale=1 1 1; visual mesh filename=package://axioma_urdf/meshes/visual/llanta.stl scale=1 1 1
- link wheel_3: geometry collision mesh filename=package://axioma_urdf/meshes/collision/llanta.dae scale=1 1 1; visual mesh filename=package://axioma_urdf/meshes/visual/llanta.stl scale=1 1 1
- link wheel_4: geometry collision mesh filename=package://axioma_urdf/meshes/collision/llanta.dae scale=1 1 1; visual mesh filename=package://axioma_urdf/meshes/visual/llanta.stl scale=1 1 1
Joints:
- joint base_to_wheel1: origin xyz=0.06442 0.07385 0.04068 rpy=3.141516 0 0 -> xyz=0.06442 0.07385 0.04068 rpy=0 0 0
- joint base_to_wheel2: origin xyz=-0.071224 0.07385 0.04068 rpy=3.141516 0 0 -> xyz=-0.071224 0.07385 0.04068 rpy=0 0 0
- joint base_to_wheel3: axis 0 -1 0 -> 0 1 0; origin xyz=-0.071224 -0.0625 0.04068 rpy=0 0 0 -> xyz=-0.071224 -0.0625 0.04068 rpy=0 0 -3.14159
- joint base_to_wheel4: axis 0 -1 0 -> 0 1 0; origin xyz=0.064423 -0.0625 0.04068 rpy=0 0 0 -> xyz=0.064423 -0.0625 0.04068 rpy=0 0 -3.14159
